Commit message: [08,09] moving grasp to 09

File: common_packages/src/ur_description/urdf/ur10.urdf.xacro (robot description, xacro)
@@ -1,67 +1,60 @@
 <?xml version="1.0"?>
 <robot xmlns:xacro="http://wiki.ros.org/xacro">
-<!--
+  <!--
   Author: Kelsey Hawkins
   Contributers: Jimmy Da Silva, Ajit Krisshna N L, Muhammad Asif Rana
 -->
-  <xacro:include filename="$(find ur_description)/urdf/ur.transmission.xacro" />
-  <xacro:include filename="$(find ur_description)/urdf/ur.gazebo.xacro" />
+  <xacro:include filename="$(find ur_description)/urdf/ur.transmission.xacro"/>
+  <xacro:include filename="$(find ur_description)/urdf/ur.gazebo.xacro"/>
   <xacro:macro name="cylinder_inertial" params="radius length mass *origin">
     <inertial>
-      <mass value="${mass}" />
-      <xacro:insert_block name="origin" />
-      <inertia ixx="${0.0833333 * mass * (3 * radius * radius + length * length)}" ixy="0.0" ixz="0.0"
-        iyy="${0.0833333 * mass * (3 * radius * radius + length * length)}" iyz="0.0"
-        izz="${0.5 * mass * radius * radius}" />
+      <mass value="${mass}"/>
+      <xacro:insert_block name="origin"/>
+      <inertia ixx="${0.0833333 * mass * (3 * radius * radius + length * length)}" ixy="0.0" ixz="0.0" iyy="${0.0833333 * mass * (3 * radius * radius + length * length)}" iyz="0.0" izz="${0.5 * mass * radius * radius}"/>
     </inertial>
   </xacro:macro>
-  <xacro:macro name="ur10_robot" params="prefix joint_limited
-    shoulder_pan_lower_limit:=${-pi}    shoulder_pan_upper_limit:=${pi}
-    shoulder_lift_lower_limit:=${-pi}    shoulder_lift_upper_limit:=${pi}
-    elbow_joint_lower_limit:=${-pi}    elbow_joint_upper_limit:=${pi}
-    wrist_1_lower_limit:=${-pi}    wrist_1_upper_limit:=${pi}
-    wrist_2_lower_limit:=${-pi}    wrist_2_upper_limit:=${pi}
-    wrist_3_lower_limit:=${-pi}    wrist_3_upper_limit:=${pi}
-    transmission_hw_interface:=hardware_interface/PositionJointInterface
-    safety_limits:=false safety_pos_margin:=0.15
-    safety_k_position:=20">
+  <xacro:macro name="ur10_robot" params="prefix joint_limited     shoulder_pan_lower_limit:=${-pi}    shoulder_pan_upper_limit:=${pi}     shoulder_lift_lower_limit:=${-pi}    shoulder_lift_upper_limit:=${pi}     elbow_joint_lower_limit:=${-pi}    elbow_joint_upper_limit:=${pi}     wrist_1_lower_limit:=${-pi}    wrist_1_upper_limit:=${pi}     wrist_2_lower_limit:=${-pi}    wrist_2_upper_limit:=${pi}     wrist_3_lower_limit:=${-pi}    wrist_3_upper_limit:=${pi}     transmission_hw_interface:=hardware_interface/PositionJointInterface     safety_limits:=false safety_pos_margin:=0.15     safety_k_position:=20">
     <!-- Inertia parameters -->
-    <xacro:property name="base_mass" value="4.0" />  <!-- This mass might be incorrect -->
-    <xacro:property name="shoulder_mass" value="7.778" />
-    <xacro:property name="upper_arm_mass" value="12.93" />
-    <xacro:property name="forearm_mass" value="3.87" />
-    <xacro:property name="wrist_1_mass" value="1.96" />
-    <xacro:property name="wrist_2_mass" value="1.96" />
-    <xacro:property name="wrist_3_mass" value="0.202" />
+    <xacro:property name="base_mass" value="4.0"/>
+    <!-- This mass might be incorrect -->
+    <xacro:property name="shoulder_mass" value="7.778"/>
+    <xacro:property name="upper_arm_mass" value="12.93"/>
+    <xacro:property name="forearm_mass" value="3.87"/>
+    <xacro:property name="wrist_1_mass" value="1.96"/>
+    <xacro:property name="wrist_2_mass" value="1.96"/>
+    <xacro:property name="wrist_3_mass" value="0.202"/>
     <!-- These parameters are borrowed from the urcontrol.conf file
         but are not verified for the correct permutation.
         The permutation was guessed by looking at the UR5 parameters.
         Serious use of these parameters needs further inspection. -->
-    <xacro:property name="shoulder_cog" value="0.00008 0.00244 -0.037" />
-    <xacro:property name="upper_arm_cog" value="0.00001 0.15061 0.38757" />
-    <xacro:property name="forearm_cog" value="-0.00012 0.06112 0.1984" />
-    <xacro:property name="wrist_1_cog" value="-0.00021 -0.00112 0.02269" />
-    <xacro:property name="wrist_2_cog" value="-0.00021 0.00112 0.002269" />
-    <xacro:property name="wrist_3_cog" value="0 -0.001156 -0.00149" />
+    <xacro:property name="shoulder_cog" value="0.00008 0.00244 -0.037"/>
+    <xacro:property name="upper_arm_cog" value="0.00001 0.15061 0.38757"/>
+    <xacro:property name="forearm_cog" value="-0.00012 0.06112 0.1984"/>
+    <xacro:property name="wrist_1_cog" value="-0.00021 -0.00112 0.02269"/>
+    <xacro:property name="wrist_2_cog" value="-0.00021 0.00112 0.002269"/>
+    <xacro:property name="wrist_3_cog" value="0 -0.001156 -0.00149"/>
     <!-- Kinematic model -->
     <!-- Properties from urcontrol.conf -->
-    <xacro:property name="d1" value="0.1273" />
-    <xacro:property name="a2" value="-0.612" />
-    <xacro:property name="a3" value="-0.5723" />
-    <xacro:property name="d4" value="0.163941" />
-    <xacro:property name="d5" value="0.1157" />
-    <xacro:property name="d6" value="0.0922" />
+    <xacro:property name="d1" value="0.1273"/>
+    <xacro:property name="a2" value="-0.612"/>
+    <xacro:property name="a3" value="-0.5723"/>
+    <xacro:property name="d4" value="0.163941"/>
+    <xacro:property name="d5" value="0.1157"/>
+    <xacro:property name="d6" value="0.0922"/>
     <!-- Arbitrary offsets for shoulder/elbow joints -->
-    <xacro:property name="shoulder_offset" value="0.220941" />  <!-- measured from model -->
-    <xacro:property name="elbow_offset" value="-0.1719" /> <!-- measured from model -->
-    <xacro:property name="upper_arm_inertia_offset" value="0.045" />  <!-- measured from model -->
+    <xacro:property name="shoulder_offset" value="0.220941"/>
+    <!-- measured from model -->
+    <xacro:property name="elbow_offset" value="-0.1719"/>
+    <!-- measured from model -->
+    <xacro:property name="upper_arm_inertia_offset" value="0.045"/>
+    <!-- measured from model -->
     <!-- link lengths used in model -->
-    <xacro:property name="shoulder_height" value="${d1}" />
-    <xacro:property name="upper_arm_length" value="${-a2}" />
-    <xacro:property name="forearm_length" value="${-a3}" />
-    <xacro:property name="wrist_1_length" value="${d4 - elbow_offset - shoulder_offset}" />
-    <xacro:property name="wrist_2_length" value="${d5}" />
-    <xacro:property name="wrist_3_length" value="${d6}" />
-    <link name="${prefix}base_link" >
+    <xacro:property name="shoulder_height" value="${d1}"/>
+    <xacro:property name="upper_arm_length" value="${-a2}"/>
+    <xacro:property name="forearm_length" value="${-a3}"/>
+    <xacro:property name="wrist_1_length" value="${d4 - elbow_offset - shoulder_offset}"/>
+    <xacro:property name="wrist_2_length" value="${d5}"/>
+    <xacro:property name="wrist_3_length" value="${d6}"/>
+    <link name="${prefix}base_link">
       <visual>
         <geometry>
@@ -78,12 +71,12 @@
       </collision>
       <xacro:cylinder_inertial radius="0.075" length="0.038" mass="${base_mass}">
-        <origin xyz="0.0 0.0 0.0" rpy="0 0 0" />
+        <origin xyz="0.0 0.0 0.0" rpy="0 0 0"/>
       </xacro:cylinder_inertial>
     </link>
     <joint name="${prefix}shoulder_pan_joint" type="revolute">
-      <parent link="${prefix}base_link" />
-      <child link = "${prefix}shoulder_link" />
-      <origin xyz="0.0 0.0 ${shoulder_height}" rpy="0.0 0.0 0.0" />
-      <axis xyz="0 0 1" />
+      <parent link="${prefix}base_link"/>
+      <child link="${prefix}shoulder_link"/>
+      <origin xyz="0.0 0.0 ${shoulder_height}" rpy="0.0 0.0 0.0"/>
+      <axis xyz="0 0 1"/>
       <xacro:unless value="${joint_limited}">
         <limit lower="${-2.0 * pi}" upper="${2.0 * pi}" effort="330.0" velocity="2.16"/>
@@ -98,5 +91,5 @@
         </xacro:if>
       </xacro:if>
-      <dynamics damping="0.0" friction="0.0"/>
+      <dynamics damping="0.01" friction="0.0"/>
     </joint>
     <link name="${prefix}shoulder_link">
@@ -115,12 +108,12 @@
       </collision>
       <xacro:cylinder_inertial radius="0.075" length="0.178" mass="${shoulder_mass}">
-        <origin xyz="0.0 0.0 0.0" rpy="0 0 0" />
+        <origin xyz="0.0 0.0 0.0" rpy="0 0 0"/>
       </xacro:cylinder_inertial>
     </link>
     <joint name="${prefix}shoulder_lift_joint" type="revolute">
-      <parent link="${prefix}shoulder_link" />
-      <child link = "${prefix}upper_arm_link" />
-      <origin xyz="0.0 ${shoulder_offset} 0.0" rpy="0.0 ${pi / 2.0} 0.0" />
-      <axis xyz="0 1 0" />
+      <parent link="${prefix}shoulder_link"/>
+      <child link="${prefix}upper_arm_link"/>
+      <origin xyz="0.0 ${shoulder_offset} 0.0" rpy="0.0 ${pi / 2.0} 0.0"/>
+      <axis xyz="0 1 0"/>
       <xacro:unless value="${joint_limited}">
         <limit lower="${-2.0 * pi}" upper="${2.0 * pi}" effort="330.0" velocity="2.16"/>
@@ -135,5 +128,5 @@
         </xacro:if>
       </xacro:if>
-      <dynamics damping="0.0" friction="0.0"/>
+      <dynamics damping="0.01" friction="0.0"/>
     </joint>
     <link name="${prefix}upper_arm_link">
@@ -152,12 +145,12 @@
       </collision>
       <xacro:cylinder_inertial radius="0.075" length="${-a2}" mass="${upper_arm_mass}">
-        <origin xyz="0.0 ${-upper_arm_inertia_offset} ${-a2/2.0}" rpy="0 0 0" />
+        <origin xyz="0.0 ${-upper_arm_inertia_offset} ${-a2/2.0}" rpy="0 0 0"/>
       </xacro:cylinder_inertial>
     </link>
     <joint name="${prefix}elbow_joint" type="revolute">
-      <parent link="${prefix}upper_arm_link" />
-      <child link = "${prefix}forearm_link" />
-      <origin xyz="0.0 ${elbow_offset} ${upper_arm_length}" rpy="0.0 0.0 0.0" />
-      <axis xyz="0 1 0" />
+      <parent link="${prefix}upper_arm_link"/>
+      <child link="${prefix}forearm_link"/>
+      <origin xyz="0.0 ${elbow_offset} ${upper_arm_length}" rpy="0.0 0.0 0.0"/>
+      <axis xyz="0 1 0"/>
       <xacro:unless value="${joint_limited}">
         <limit lower="${-pi}" upper="${pi}" effort="150.0" velocity="3.15"/>
@@ -172,9 +165,9 @@
         </xacro:if>
       </xacro:if>
-      <dynamics damping="0.0" friction="0.0"/>
+      <dynamics damping="0.01" friction="0.0"/>
     </joint>
     <link name="${prefix}forearm_link">
       <visual>
-         <geometry>
+        <geometry>
           <mesh filename="package://ur_description/meshes/ur10/visual/forearm.dae"/>
         </geometry>
@@ -189,12 +182,12 @@
       </collision>
       <xacro:cylinder_inertial radius="0.075" length="${-a3}" mass="${forearm_mass}">
-        <origin xyz="0.0 0.0 ${-a3/2.0}" rpy="0 0 0" />
+        <origin xyz="0.0 0.0 ${-a3/2.0}" rpy="0 0 0"/>
       </xacro:cylinder_inertial>
     </link>
     <joint name="${prefix}wrist_1_joint" type="revolute">
-      <parent link="${prefix}forearm_link" />
-      <child link = "${prefix}wrist_1_link" />
-      <origin xyz="0.0 0.0 ${forearm_length}" rpy="0.0 ${pi / 2.0} 0.0" />
-      <axis xyz="0 1 0" />
+      <parent link="${prefix}forearm_link"/>
+      <child link="${prefix}wrist_1_link"/>
+      <origin xyz="0.0 0.0 ${forearm_length}" rpy="0.0 ${pi / 2.0} 0.0"/>
+      <axis xyz="0 1 0"/>
       <xacro:unless value="${joint_limited}">
         <limit lower="${-2.0 * pi}" upper="${2.0 * pi}" effort="54.0" velocity="3.2"/>
@@ -209,5 +202,5 @@
         </xacro:if>
       </xacro:if>
-      <dynamics damping="0.0" friction="0.0"/>
+      <dynamics damping="0.01" friction="0.0"/>
     </joint>
     <link name="${prefix}wrist_1_link">
@@ -226,12 +219,12 @@
       </collision>
       <xacro:cylinder_inertial radius="0.075" length="0.12" mass="${wrist_1_mass}">
-        <origin xyz="0.0 ${wrist_1_length} 0.0" rpy="0 0 0" />
+        <origin xyz="0.0 ${wrist_1_length} 0.0" rpy="0 0 0"/>
       </xacro:cylinder_inertial>
     </link>
     <joint name="${prefix}wrist_2_joint" type="revolute">
-      <parent link="${prefix}wrist_1_link" />
-      <child link = "${prefix}wrist_2_link" />
-      <origin xyz="0.0 ${wrist_1_length} 0.0" rpy="0.0 0.0 0.0" />
-      <axis xyz="0 0 1" />
+      <parent link="${prefix}wrist_1_link"/>
+      <child link="${prefix}wrist_2_link"/>
+      <origin xyz="0.0 ${wrist_1_length} 0.0" rpy="0.0 0.0 0.0"/>
+      <axis xyz="0 0 1"/>
       <xacro:unless value="${joint_limited}">
         <limit lower="${-2.0 * pi}" upper="${2.0 * pi}" effort="54.0" velocity="3.2"/>
@@ -246,5 +239,5 @@
         </xacro:if>
       </xacro:if>
-      <dynamics damping="0.0" friction="0.0"/>
+      <dynamics damping="0.01" friction="0.0"/>
     </joint>
     <link name="${prefix}wrist_2_link">
@@ -263,12 +256,12 @@
       </collision>
       <xacro:cylinder_inertial radius="0.075" length="0.12" mass="${wrist_2_mass}">
-        <origin xyz="0.0 0.0 ${wrist_2_length}" rpy="0 0 0" />
+        <origin xyz="0.0 0.0 ${wrist_2_length}" rpy="0 0 0"/>
       </xacro:cylinder_inertial>
     </link>
     <joint name="${prefix}wrist_3_joint" type="revolute">
-      <parent link="${prefix}wrist_2_link" />
-      <child link = "${prefix}wrist_3_link" />
-      <origin xyz="0.0 0.0 ${wrist_2_length}" rpy="0.0 0.0 0.0" />
-      <axis xyz="0 1 0" />
+      <parent link="${prefix}wrist_2_link"/>
+      <child link="${prefix}wrist_3_link"/>
+      <origin xyz="0.0 0.0 ${wrist_2_length}" rpy="0.0 0.0 0.0"/>
+      <axis xyz="0 1 0"/>
       <xacro:unless value="${joint_limited}">
         <limit lower="${-2.0 * pi}" upper="${2.0 * pi}" effort="54.0" velocity="3.2"/>
@@ -283,5 +276,5 @@
         </xacro:if>
       </xacro:if>
-      <dynamics damping="0.0" friction="0.0"/>
+      <dynamics damping="0.01" friction="0.0"/>
     </joint>
     <link name="${prefix}wrist_3_link">
@@ -300,11 +293,11 @@
       </collision>
       <xacro:cylinder_inertial radius="0.045" length="0.0305" mass="${wrist_3_mass}">
-        <origin xyz="0.0 ${wrist_3_length - 0.0305/2} 0.0" rpy="${pi/2} 0 0" />
+        <origin xyz="0.0 ${wrist_3_length - 0.0305/2} 0.0" rpy="${pi/2} 0 0"/>
       </xacro:cylinder_inertial>
     </link>
     <joint name="${prefix}ee_fixed_joint" type="fixed">
-      <parent link="${prefix}wrist_3_link" />
-      <child link = "${prefix}ee_link" />
-      <origin xyz="0.0 ${wrist_3_length} 0.0" rpy="0.0 0.0 ${pi/2.0}" />
+      <parent link="${prefix}wrist_3_link"/>
+      <child link="${prefix}ee_link"/>
+      <origin xyz="0.0 ${wrist_3_length} 0.0" rpy="0.0 0.0 ${pi/2.0}"/>
     </joint>
     <link name="${prefix}ee_link">
@@ -316,6 +309,6 @@
       </collision>
     </link>
-    <xacro:ur_arm_transmission prefix="${prefix}" hw_interface="${transmission_hw_interface}" />
-    <xacro:ur_arm_gazebo prefix="${prefix}" />
+    <xacro:ur_arm_transmission prefix="${prefix}" hw_interface="${transmission_hw_interface}"/>
+    <xacro:ur_arm_gazebo prefix="${prefix}"/>
     <!-- ROS base_link to UR 'Base' Coordinates transform -->
     <link name="${prefix}base"/>
