Commit message: [09] urdf2collision good point, tools upgraded

File: 09_manipulation/src/moveit_grasps/moveit_grasp_b_tools/urdf/box.urdf (robot description, URDF)
Before this commit: robot materials, 1 links, 0 joints
Links:
- link base_link: geometry visual box size=0.05 0.05 0.08

File: 09_manipulation/src/moveit_grasps/moveit_grasp_b_tools/urdf/cilinder.urdf (robot description, URDF)
Before this commit: robot materials, 1 links, 0 joints
Links:
- link base_link: geometry visual cylinder length=0.04 radius=0.04
