Commit message: [09] testing urdf to colision object

File: 09_manipulation/src/moveit_grasps/moveit_grasp_b_tools/urdf/test.urdf (robot description, URDF)
Before this commit: robot physics, 16 links, 15 joints
Joints:
- joint gripper_extension: type prismatic -> fixed
- joint head_swivel: type continuous -> fixed
- joint left_back_wheel_joint: type continuous -> fixed
- joint left_front_wheel_joint: type continuous -> fixed
- joint left_gripper_joint: type revolute -> fixed
- joint right_back_wheel_joint: type continuous -> fixed
- joint right_front_wheel_joint: type continuous -> fixed
- joint right_gripper_joint: type revolute -> fixed

Commit message: [09] testing urdf to colision object

File: 09_manipulation/src/moveit_grasps/moveit_grasp_b_tools/urdf/test.urdf (robot description, URDF)
Before this commit: robot physics, 16 links, 15 joints
Links:
- removed link box
- removed link gripper_pole
- removed link head
- removed link left_back_wheel
- removed link left_base
- removed link left_front_wheel
- removed link left_gripper
- removed link left_tip
- removed link right_back_wheel
- removed link right_base
- removed link right_front_wheel
- removed link right_gripper
- removed link right_tip
- link base_link: mass 10 -> None; geometry visual cylinder length=0.6 radius=0.2
- link left_leg: mass 10 -> None; geometry visual box size=0.6 0.1 0.2
- link right_leg: mass 10 -> None; geometry visual box size=0.6 0.1 0.2
Joints:
- removed joint gripper_extension
- removed joint head_swivel
- removed joint left_back_wheel_joint
- removed joint left_base_joint
- removed joint left_front_wheel_joint
- removed joint left_gripper_joint
- removed joint left_tip_joint
- removed joint right_back_wheel_joint
- removed joint right_base_joint
- removed joint right_front_wheel_joint
- removed joint right_gripper_joint
- removed joint right_tip_joint
- removed joint tobox

Commit message: [*] wip

File: 09_manipulation/src/moveit_grasps/moveit_grasp_b_tools/urdf/test.urdf (robot description, URDF)
Before this commit: robot materials, 1 links, 0 joints
Links:
- link base_link: geometry visual cylinder length=0.1 radius=0.02
