Commit message: [common] create moveit conf pack for robot with gripper

File: common_packages/src/workspace_description/urdf/robot_with_gripper.xacro (robot description, xacro)
@@ -9,5 +9,4 @@
   <xacro:include filename="$(find ur_description)/urdf/ur10.urdf.xacro"/>
   <xacro:include filename="$(find robotiq_85_description)/urdf/robotiq_85_gripper.urdf.xacro"/>
-  <xacro:include filename="$(find smart_app_ur_station_description)/urdf/station.xacro"/>
   <!-- 3. Place ur3 robot and attach it to gazebo station_base-->
   <!-- 3.1 declare load kinematics and transmission info-->
@@ -36,21 +35,4 @@
     <origin xyz="0 0 0" rpy="0 0 0"/>
   </joint>
-  <link name="end_effector">
-    <visual>
-      <geometry>
-        <box size="0.01 0.01 0.01"/>
-      </geometry>
-    </visual>
-    <collision>
-      <geometry>
-        <box size="0.01 0.01 0.01"/>
-      </geometry>
-    </collision>
-  </link>
-  <joint name="world_joint" type="fixed">
-    <parent link="station_base"/>
-    <child link="base_link"/>
-    <origin xyz="0.0 0.0 0.7" rpy="0.0 0.0 0.0"/>
-  </joint>
   <!-- 4. Place the wripper attached to the UR10 frame called tool0 -->
   <xacro:robotiq_85_gripper prefix="" parent="tool0">
@@ -58,4 +40,3 @@
   </xacro:robotiq_85_gripper>
   <!-- 5. Place the Table-->
-  <xacro:table xyz="-0.029 0.335 0.630" connected_to="station_base"/>
 </robot>
